File: outputs/pcbs/keeb_left.kicad_pcb (KiCad board)
At the start: 2 copper layers, 135.4 x 117 mm, 70 parts

Commit message: Adding latest outputs from ergogen
Parts:
- removed XX1: , SW-TH_K3-1235S-L1
- removed XX2: , easyeda2kicad:CONN-SMD_1.25T-2P-WT
- added JST1: , CONN-SMD_1.25T-2P-WT, B.Cu at (196.3, 160.9)
- added PWR1: , SW-TH_K3-1235D-L1, F.Cu at (156.0, 169.4)
- RST1: footprint easyeda2kicad:KEY-SMD_L6.0-W3.3-LS6.7 -> KEY-SMD_L6.0-W3.3-LS6.7
- moved RST1 1.00 mm to (175.2, 177.3)
- moved MCU1 0.53 mm to (173.2, 141.9)
Other:
- outline, holes or cut-outs redrawn
