File: outputs/pcbs/keeb_right.kicad_pcb (KiCad board)
At the start: 2 copper layers, 135.4 x 117 mm, 70 parts

Commit message: Adding latest outputs from ergogen
Parts:
- removed XX1: , SW-TH_K3-1235S-L1
- removed XX2: , easyeda2kicad:CONN-SMD_1.25T-2P-WT
- added JST1: , CONN-SMD_1.25T-2P-WT, B.Cu at (239.9, 160.9)
- added PWR1: , SW-TH_K3-1235D-L1, F.Cu at (280.2, 169.4)
- RST1: footprint easyeda2kicad:KEY-SMD_L6.0-W3.3-LS6.7 -> KEY-SMD_L6.0-W3.3-LS6.7
- moved RST1 1.00 mm to (261.1, 177.3)
- moved MCU1 0.53 mm to (263.0, 141.9)
Connections:
- D1 pad 1: P8 -> P9
- D10 pad 1: P4 -> P6
- D11 pad 1: P8 -> P9
- D13 pad 1: P6 -> P4
- D15 pad 1: P4 -> P6
- D16 pad 1: P8 -> P9
- D18 pad 1: P6 -> P4
- D20 pad 1: P4 -> P6
- D22 pad 1: P4 -> P6
- D24 pad 1: P4 -> P6
- D25 pad 1: P6 -> P4
- D27 pad 1: P4 -> P6
- D3 pad 1: P6 -> P4
- D30 pad 1: P6 -> P4
- D32 pad 1: P6 -> P4
- D5 pad 1: P4 -> P6
- D6 pad 1: P8 -> P9
- D8 pad 1: P6 -> P4
- RST1 pad 1: GND -> RST
- RST1 pad 2: RST -> GND
Other:
- outline, holes or cut-outs redrawn
